File: hardware/baseBoard/baseBoard.sch (KiCad schematic (older format))
At the start: 32 parts, among them J1 Screw_Terminal_01x06, J2 Conn_01x03, J3 Conn_01x06, Q1 BC817, U1 Finder66.22, U2 MCP601-xOT, U3 CS1XXX, U4 AP65111AWU

Commit message: sch / pcb update
Parts:
- removed U2: MCP601-xOT, Package_TO_SOT_SMD:SOT-23-5, symbol Amplifier_Operational:MCP601-xOT
- added H1, H2, H3, H4, H5: MountingHole, MountingHole:MountingHole_4.3mm_M4, symbol Mechanical:MountingHole
- added J4, J5: Conn_01x01, Connector_Pin:Pin_D1.4mm_L8.5mm_W2.8mm_FlatFork, symbol Connector_Generic:Conn_01x01
- added R12: tbd, Resistor_SMD:R_0603_1608Metric, symbol Device:R
- added U2: MCP6L02x-xSN, Package_SO:SOIC-8_3.9x4.9mm_P1.27mm, symbol Amplifier_Operational:MCP6L02x-xSN
- J2: footprint (none) -> Connector_Phoenix_MC:PhoenixContact_MCV_1,5_3-G-3.81_1x03_P3.81mm_Vertical
- J3: footprint (none) -> baseBoard:2178710-6
- R6: value tbd -> 75k
Connections:
- net +5V: now also U2.8 (V+)
- net C_SENS: now also U2.1
- net GND: now also U2.4 (V-)
- net L: now also J5.1 (Pin_1); no longer U1.21
- net L_MOTOR: now also U1.14; no longer U1.24
- net N: now also U1.21; no longer U1.11
- net N_MOTOR: now also U1.24; no longer U1.14
- net at R7.2, U3.1: now also R12.2
- net at R5.1, R6.2: now also U2.5 (+); no longer U3.3
- net at C5.1, R7.1: now also U2.3 (+)
- net at R8.2, R9.2: now also U2.2 (-)
- new net: J4.1 (Pin_1), U1.11
- new net: R12.1, U2.6 (-), U2.7, U3.3
Other:
- moved on the sheet: C5, C6, R5, R6, R7, R8, R9, U3
